File: MainBoard/DiscreteComparator.kicad_sch (KiCad schematic)
At the start: 22 parts, among them Q17 BC557, Q18 BC557, Q19 BC557, Q20 BC557, Q21 BC557, Q22 BC557, Q23 BC557, Q24 BC557, Q25 BC557, Q26 BC547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

Commit message: functional -- but very slow slew rates
Connections:
- net -v: no longer Q22.1 (C), Q30.1 (C), Q30.2 (B), Q31.2 (B)
- new net: Q22.1 (C), Q30.1 (C), Q30.2 (B), Q31.2 (B)
Changed lines of the file:
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@@
-	(hierarchical_label "-v"
-		(shape input)
-		(at 119.38 102.87 270)
-		(effects
-			(font
-				(size 1.27 1.27)
-			)
-			(justify right)
-		)
-	)
 	(hierarchical_label "-v"
 		(shape input)

Commit message: WIP
Other:
- moved on the sheet: RV3
Changed lines of the file:
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@@
 	(wire
 		(pts
-			(xy 67.31 59.69) (xy 67.31 62.23)
+			(xy 67.31 58.42) (xy 67.31 60.96)
 		)
 		(stroke
@@
 	(wire
 		(pts
-			(xy 67.31 69.85) (xy 67.31 72.39)
+			(xy 67.31 68.58) (xy 67.31 71.12)
 		)
 		(stroke
@@
 	(wire
 		(pts
-			(xy 71.12 66.04) (xy 73.66 66.04)
+			(xy 71.12 64.77) (xy 73.66 64.77)
 		)
 		(stroke
@@
 	)
 	(label "InternalBias"
-		(at 73.66 66.04 0)
+		(at 73.66 64.77 0)
 		(effects
 			(font
@@
 	(hierarchical_label "+v"
 		(shape input)
-		(at 67.31 59.69 90)
+		(at 67.31 58.42 90)
 		(effects
 			(font
@@
 	(symbol
 		(lib_id "power:GND")
-		(at 67.31 72.39 0)
+		(at 67.31 71.12 0)
 		(unit 1)
 		(exclude_from_sim no)
@@
 		(dnp no)
 		(property "Reference" "#PWR010"
-			(at 67.31 78.74 0)
+			(at 67.31 77.47 0)
 			(effects
 				(font
@@
 		)
 		(property "Value" "GND"
-			(at 67.31 76.2 0)
+			(at 67.31 74.93 0)
 			(effects
 				(font
@@
 		)
 		(property "Footprint" ""
-			(at 67.31 72.39 0)
+			(at 67.31 71.12 0)
 			(effects
 				(font
@@
 		)
 		(property "Datasheet" ""
-			(at 67.31 72.39 0)
+			(at 67.31 71.12 0)
 			(effects
 				(font
@@
 		)
 		(property "Description" "Power symbol creates a global label with name \"GND\" , ground"
-			(at 67.31 72.39 0)
+			(at 67.31 71.12 0)
 			(effects
 				(font
@@
 	(symbol
 		(lib_id "Device:R_Potentiometer_Trim")
-		(at 67.31 66.04 0)
+		(at 67.31 64.77 0)
 		(unit 1)
 		(exclude_from_sim no)
@@
 		(fields_autoplaced yes)
 		(property "Reference" "RV3"
-			(at 64.77 64.7699 0)
+			(at 64.77 63.4999 0)
 			(effects
 				(font
@@
 		)
 		(property "Value" "10k"
-			(at 64.77 67.3099 0)
+			(at 64.77 66.0399 0)
 			(effects
 				(font
@@
 		)
 		(property "Footprint" "Potentiometer_THT:Potentiometer_TT_P0915N"
-			(at 67.31 66.04 0)
+			(at 67.31 64.77 0)
 			(effects
 				(font
@@
 		)
 		(property "Datasheet" "~"
-			(at 67.31 66.04 0)
+			(at 67.31 64.77 0)
 			(effects
 				(font
@@
 		)
 		(property "Description" "Trim-potentiometer"
-			(at 67.31 66.04 0)
+			(at 67.31 64.77 0)
 			(effects
 				(font
@@
 		)
 		(property "Sim.Library" "models/potentiometer.lib"
-			(at 67.31 66.04 0)
+			(at 67.31 64.77 0)
 			(effects
 				(font
@@
 		)
 		(property "Sim.Name" "POT"
-			(at 67.31 66.04 0)
+			(at 67.31 64.77 0)
 			(effects
 				(font
@@
 		)
 		(property "Sim.Device" "SUBCKT"
-			(at 67.31 66.04 0)
+			(at 67.31 64.77 0)
 			(effects
 				(font
@@
 		)
 		(property "Sim.Pins" "1=1 2=2 3=3"
-			(at 67.31 66.04 0)
+			(at 67.31 64.77 0)
 			(effects
 				(font
@@
 		)
 		(property "Sim.Params" "Rtot=10k w=0.3"
-			(at 67.31 66.04 0)
-			(effects
-				(font
+			(at 67.31 64.77 0)
+			(effects
+				(font

Commit message: WIP: trying to fix internal bias
Parts:
- added C1: 10u, Capacitor_THT:C_Rect_L9.0mm_W2.5mm_P7.50mm_MKT, symbol Device:C
- added C3: 100n, Capacitor_THT:C_Rect_L9.0mm_W2.5mm_P7.50mm_MKT, symbol Device:C
- added Q16: BC557, Package_TO_SOT_THT:TO-92_Inline, symbol Transistor_BJT:BC557
- added R1: 1M, Resistor_THT:R_Axial_DIN0207_L6.3mm_D2.5mm_P7.62mm_Horizontal, symbol Device:R
- C6: value 1n -> 100p
- R6: value 100k -> 1M
Connections:
- net -v: now also R1.1
- net GND: now also C1.2, C3.2
- net InternalBias: now also Q16.3 (E); no longer RV3.2
- new net: C1.1, C3.1, Q16.2 (B), RV3.2
- new net: Q16.1 (C), R1.2
Other:
- moved on the sheet: RV3

Commit message: stiffing of internal bias
Parts:
- removed Q27: BC557, Package_TO_SOT_THT:TO-92_Inline, symbol Transistor_BJT:BC557
- added C7: 10u, Capacitor_THT:C_Rect_L9.0mm_W2.5mm_P7.50mm_MKT, symbol Device:C
- added Q11: BC557, Package_TO_SOT_THT:TO-92_Inline, symbol Transistor_BJT:BC557
- added R11: 100, Resistor_THT:R_Axial_DIN0207_L6.3mm_D2.5mm_P7.62mm_Horizontal, symbol Device:R
- added R13: 1k, Resistor_THT:R_Axial_DIN0207_L6.3mm_D2.5mm_P7.62mm_Horizontal, symbol Device:R
- C1: value 10u -> 100u
- R1: value 1M -> 10k
Connections:
- net GND is gone; now on net -v: C1.2, C3.2, RV3.3
- net -v: now also C7.2
- net InternalBias: now also C7.1, Q11.2 (B), R11.1; no longer Q16.3 (E)
- net at D15.1 (K), D17.1 (K), Q22.2 (B): now also R13.2; no longer Q24.3 (E)
- net at Q18.1 (C), Q22.3 (E), Q23.3 (E): now also Q11.3 (E)
- net at Q23.1 (C), Q29.2 (B), Q31.1 (C): now also Q11.1 (C)
- new net: Q24.3 (E), R13.1
- new net: Q16.3 (E), R11.2
Other:
- note added: "Common-mode Voltage Clamp"
- note removed: "Common-mode voltage clamp"
- moved on the sheet: C1, C3, Q16, Q24, R1, RV3
